File: schematics/GroBot.sch (KiCad schematic (older format))
At the start: 43 parts

Commit message: Change the water temp resistor value.
Fixes #10
Parts:
- R?: value 12k -> 30k
Changed lines of the file:
@@
 P 2550 7150
 F 0 "R?" V 2630 7150 50  0000 C CNN
-F 1 "12k" V 2550 7150 50  0000 C CNN
+F 1 "30k" V 2550 7150 50  0000 C CNN
 F 2 "" V 2480 7150 50  0000 C CNN
 F 3 "" H 2550 7150 50  0000 C CNN

Commit message: Add component for STM 32 MCU.
Fixes #11
Parts:
- added U?: STM32F091CBU6, symbol STM32F091CBU6
Other:
- note added: "ANALOG REF"
Changed lines of the file:
@@
 LIBS:valves
 LIBS:psoc
+LIBS:stm
 LIBS:GroBot-cache
 EELAYER 25 0
@@
 Connection ~ 7550 2850
 Connection ~ 8100 2850
+$Comp
+L STM32F091CBU6 U?
+U 1 1 58EAEB8D
+P 9850 3100
+F 0 "U?" H 9950 2700 60  0000 C CNN
+F 1 "STM32F091CBU6" H 9950 3000 60  0000 C CNN
+F 2 "" H 9950 2700 60  0000 C CNN
+F 3 "" H 9950 2700 60  0000 C CNN
+	1    9850 3100
+	1    0    0    -1
+$EndComp
+Text Notes 3300 1900 0    60   ~ 0
+ANALOG REF
 $EndSCHEMATC

Commit message: Add power regulator and supply for MCU.
This is a 3.3 V for the MCU.
Parts:
- added C?: 2.2 uF, symbol C
- added C?: 22 uF, symbol C
- added C? (x3): 100 nF, symbol C
- added C?: 10 nF, symbol C
- added C?: 1 uF, symbol C
- added C? (x2): 4.7 uF, symbol C
- added L?: 10 uH, symbol L_Small
- added R?: 100k, symbol R
- added U?: TPS62177DQCR, symbol TPS62177DQCR
Connections:
- net labels added: 3.3V, 3.3_PG, SLEEP
- wire segments 108 -> 158
Other:
- note added: "3.3 V REGULATOR"

Commit message: Add oscillator to board design.
This is an external 32 Mhz crystal for the MCU. It might not
be necessary in a final design, but it's nice to have for testing
purposes.
Parts:
- added C? (x2): 27 pF, symbol C
- added Y?: Crystal, symbol Crystal
Connections:
- wire segments 158 -> 166
Changed lines of the file:
@@
 L GND #PWR?
 U 1 1 58EBFD4C
-P 6150 8700
-F 0 "#PWR?" H 6150 8450 50  0001 C CNN
-F 1 "GND" H 6150 8550 50  0000 C CNN
-F 2 "" H 6150 8700 50  0000 C CNN
-F 3 "" H 6150 8700 50  0000 C CNN
-	1    6150 8700
+P 6000 8750
+F 0 "#PWR?" H 6000 8500 50  0001 C CNN
+F 1 "GND" H 6000 8600 50  0000 C CNN
+F 2 "" H 6000 8750 50  0000 C CNN
+F 3 "" H 6000 8750 50  0000 C CNN
+	1    6000 8750
 	-1   0    0    1
 $EndComp
@@
 	6300 9450 6300 9350
 Wire Wire Line
-	7000 8850 6150 8850
-Wire Wire Line
-	6150 8850 6150 8700
+	6000 8850 7000 8850
 Wire Wire Line
 	8450 9700 8450 10350
@@
 	9600 8600 9750 8600
 Connection ~ 9750 8600
+$Comp
+L Crystal Y?
+U 1 1 58F81FD1
+P 6150 8050
+F 0 "Y?" H 6150 8200 50  0000 C CNN
+F 1 "Crystal" H 6150 7900 50  0000 C CNN
+F 2 "" H 6150 8050 50  0000 C CNN
+F 3 "535-10239-1-ND" V 5900 8100 50  0000 C CNN
+	1    6150 8050
+	0    1    1    0
+$EndComp
+Wire Wire Line
+	6400 7900 6400 8550
+Wire Wire Line
+	6400 7900 5700 7900
+Wire Wire Line
+	6150 8200 6150 8650
+$Comp
+L C C?
+U 1 1 58F822E5
+P 5700 8050
+F 0 "C?" H 5725 8150 50  0000 L CNN
+F 1 "27 pF" H 5725 7950 50  0000 L CNN
+F 2 "" H 5738 7900 50  0000 C CNN
+F 3 "" H 5700 8050 50  0000 C CNN
+	1    5700 8050
+	1    0    0    -1
+$EndComp
+$Comp
+L C C?
+U 1 1 58F8237A
+P 5950 8300
+F 0 "C?" H 5975 8400 50  0000 L CNN
+F 1 "27 pF" H 5975 8200 50  0000 L CNN
+F 2 "" H 5988 8150 50  0000 C CNN
+F 3 "" H 5950 8300 50  0000 C CNN
+	1    5950 8300
+	0    1    1    0
+$EndComp
+Wire Wire Line
+	6100 8300 6150 8300
+Connection ~ 6150 8300
+Connection ~ 6150 7900
+Wire Wire Line
+	5700 8200 5700 8450
+Wire Wire Line
+	5700 8300 5800 8300
+Connection ~ 5700 8300
+$Comp
+L GND #PWR?
+U 1 1 58F8283F
+P 5700 8450
+F 0 "#PWR?" H 5700 8200 50  0001 C CNN
+F 1 "GND" H 5700 8300 50  0000 C CNN
+F 2 "" H 5700 8450 50  0000 C CNN
+F 3 "" H 5700 8450 50  0000 C CNN
+	1    5700 8450
+	1    0    0    -1
+$EndComp
+Wire Wire Line
+	6400 8550 7000 8550
+Wire Wire Line
+	6150 8650 7000 8650
+Wire Wire Line
+	6000 8750 6000 8850
 $EndSCHEMATC

Commit message: Add external recet circuitry.
This allows you to reset manually with a button, as well as
for the CHIP to force a reset.
Parts:
- added C?: 0.1uF, symbol C
- added SW?: SW_PUSH, symbol SW_PUSH
- C?: value 22 uF -> 22uF
- C? (x3): value 100 nF -> 100nF
- C?: value 10 nF -> 10nF
- C?: value 1 uF -> 1uF
- C? (x2): value 4.7 uF -> 4.7uF
- C? (x2): value 27 pF -> 27pF
Connections:
- net labels added: RESET
- wire segments 166 -> 171
Other:
- moved on the sheet: C?, R?

Commit message: Add all UART connections.
Parts:
- added R?: 10k, symbol R
Connections:
- net labels added: BOOT0, BTL_RX, BTL_TX, CAN_RX, CAN_TX
- wire segments 171 -> 188
Changed lines of the file:
@@
 	1    0    0    -1
 $EndComp
+Wire Wire Line
+	7850 7700 7850 7400
+Wire Wire Line
+	7850 7400 8000 7400
+Wire Wire Line
+	8000 7400 8000 6700
+Text Label 8000 6700 0    60   ~ 0
+BOOT0
+$Comp
+L R R?
+U 1 1 58F8C61C
+P 7750 6850
+F 0 "R?" V 7830 6850 50  0000 C CNN
+F 1 "10k" V 7750 6850 50  0000 C CNN
+F 2 "" V 7680 6850 50  0000 C CNN
+F 3 "" H 7750 6850 50  0000 C CNN
+	1    7750 6850
+	0    1    1    0
+$EndComp
+Wire Wire Line
+	7900 6850 8000 6850
+Connection ~ 8000 6850
+$Comp
+L GND #PWR?
+U 1 1 58F8C7DB
+P 7500 6850
+F 0 "#PWR?" H 7500 6600 50  0001 C CNN
+F 1 "GND" H 7500 6700 50  0000 C CNN
+F 2 "" H 7500 6850 50  0000 C CNN
+F 3 "" H 7500 6850 50  0000 C CNN
+	1    7500 6850
+	0    1    1    0
+$EndComp
+Wire Wire Line
+	7500 6850 7600 6850
+Text Label 9200 8650 0    60   ~ 0
+BTL_RX
+Wire Wire Line
+	9200 8650 9000 8650
+Text Label 9200 8750 0    60   ~ 0
+BTL_TX
+Wire Wire Line
+	9200 8750 9000 8750
+Text Label 8850 7550 0    60   ~ 0
+SBC_TX
+Wire Wire Line
+	8850 7550 8550 7550
+Wire Wire Line
+	8550 7550 8550 7700
+Wire Wire Line
+	8450 7700 8450 7400
+Wire Wire Line
+	8450 7400 8850 7400
+Text Label 8850 7400 0    60   ~ 0
+SBC_RX
+Text Label 7750 10200 0    60   ~ 0
+LCD_TX
+Wire Wire Line
+	7750 10200 8250 10200
+Wire Wire Line
+	8250 10200 8250 9700
+Text Label 7750 10300 0    60   ~ 0
+LCD_RX
+Wire Wire Line
+	7750 10300 8350 10300
+Wire Wire Line
+	8350 10300 8350 9700
+Text Label 9200 8550 0    60   ~ 0
+CAN_RX
+Wire Wire Line
+	9200 8550 9000 8550
+Text Label 9200 8450 0    60   ~ 0
+CAN_TX
+Wire Wire Line
+	9200 8450 9000 8450
 $EndSCHEMATC

Commit message: Add CAN transceiver.
Parts:
- added C?: 100nF, symbol C
- added U?: TLE7251V, symbol TLE7251V
Connections:
- net labels added: +3.3V, CANH, CANL, CAN_STB
- wire segments 188 -> 205
Other:
- note added: "CAN TRANCEIVER"
Changed lines of the file:
@@
 LIBS:stm
 LIBS:power_reg
+LIBS:can
 LIBS:GroBot-cache
 EELAYER 25 0
@@
 	1    0    0    -1
 $EndComp
-Text Label 4050 8500 0    60   ~ 0
-3.3V
 $Comp
 L L_Small L?
@@
 Text Label 6700 8150 0    60   ~ 0
 3.3V
-Text Label 8550 10050 0    60   ~ 0
-3.3V
-Text Label 7450 7200 0    60   ~ 0
-3.3V
 $Comp
 L C C?
@@
 	1    0    0    -1
 $EndComp
-Text Label 5750 8950 0    60   ~ 0
-3.3V
 Wire Wire Line
 	6050 2050 6500 2050
@@
 Wire Wire Line
 	2700 8700 2600 8700
-Wire Wire Line
-	5750 8950 7000 8950
 Wire Wire Line
 	8550 9700 8550 10050
@@
 Wire Wire Line
 	9200 8450 9000 8450
+$Comp
+L TLE7251V U?
+U 1 1 58F9A09B
+P 12900 7850
+F 0 "U?" H 12900 7900 60  0000 C CNN
+F 1 "TLE7251V" H 12900 8100 60  0000 C CNN
+F 2 "" H 12900 7850 60  0000 C CNN
+F 3 "" H 12900 7850 60  0000 C CNN
+	1    12900 7850
+	1    0    0    -1
+$EndComp
+Text Label 11750 7550 0    60   ~ 0
+CAN_TX
+Wire Wire Line
+	11750 7550 12200 7550
+Text Label 11750 7850 0    60   ~ 0
+CAN_RX
+Wire Wire Line
+	11750 7850 12200 7850
+Wire Wire Line
+	12200 7650 11350 7650
+Wire Wire Line
+	11350 7650 11350 7950
+$Comp
+L GND #PWR?
+U 1 1 58F9ABD1
+P 11350 7950
+F 0 "#PWR?" H 11350 7700 50  0001 C CNN
+F 1 "GND" H 11350 7800 50  0000 C CNN
+F 2 "" H 11350 7950 50  0000 C CNN
+F 3 "" H 11350 7950 50  0000 C CNN
+	1    11350 7950
+	1    0    0    -1
+$EndComp
+Wire Wire Line
+	12200 7750 11500 7750
+Wire Wire Line
+	11500 7750 11500 8300
+Wire Wire Line
+	11500 8150 11750 8150
+$Comp
+L +5V #PWR?
+U 1 1 58F9B9A2
+P 11750 8150
+F 0 "#PWR?" H 11750 8000 50  0001 C CNN
+F 1 "+5V" H 11750 8290 50  0000 C CNN
+F 2 "" H 11750 8150 50  0000 C CNN
+F 3 "" H 11750 8150 50  0000 C CNN
+	1    11750 8150
+	0    1    1    0
+$EndComp
+$Comp
+L C C?
+U 1 1 58F9BA34
+P 11500 8450
+F 0 "C?" H 11525 8550 50  0000 L CNN
+F 1 "100nF" H 11525 8350 50  0000 L CNN
+F 2 "" H 11538 8300 50  0000 C CNN
+F 3 "" H 11500 8450 50  0000 C CNN
+	1    11500 8450
+	1    0    0    -1
+$EndComp
+Connection ~ 11500 8150
+$Comp
+L GND #PWR?
+U 1 1 58F9BD47
+P 11500 8700
+F 0 "#PWR?" H 11500 8450 50  0001 C CNN
+F 1 "GND" H 11500 8550 50  0000 C CNN
+F 2 "" H 11500 8700 50  0000 C CNN
+F 3 "" H 11500 8700 50  0000 C CNN
+	1    11500 8700
+	1    0    0    -1
+$EndComp
+Wire Wire Line
+	11500 8700 11500 8600
+$Comp
+L +3.3V #PWR?
+U 1 1 58F9C712
+P 4050 8500
+F 0 "#PWR?" H 4050 8350 50  0001 C CNN
+F 1 "+3.3V" H 4050 8640 50  0000 C CNN
+F 2 "" H 4050 8500 50  0000 C CNN
+F 3 "" H 4050 8500 50  0000 C CNN
+	1    4050 8500
+	0    1    1    0
+$EndComp
+Wire Wire Line
+	5800 8950 7000 8950
+$Comp
+L +3.3V #PWR?
+U 1 1 58F9CF41
+P 5800 9000
+F 0 "#PWR?" H 5800 8850 50  0001 C CNN
+F 1 "+3.3V" H 5800 9140 50  0000 C CNN
+F 2 "" H 5800 9000 50  0000 C CNN
+F 3 "" H 5800 9000 50  0000 C CNN
+	1    5800 9000
+	-1   0    0    1
+$EndComp
+Wire Wire Line
+	5800 9000 5800 8950
+$Comp
+L +3.3V #PWR?
+U 1 1 58F9D708
+P 8650 10150
+F 0 "#PWR?" H 8650 10000 50  0001 C CNN
+F 1 "+3.3V" H 8650 10290 50  0000 C CNN
+F 2 "" H 8650 10150 50  0000 C CNN
+F 3 "" H 8650 10150 50  0000 C CNN
+	1    8650 10150
+	-1   0    0    1
+$EndComp
+Wire Wire Line
+	8650 10150 8650 10050
+Wire Wire Line
+	8650 10050 8550 10050
+$Comp
+L +3.3V #PWR?
+U 1 1 58F9DD50
+P 7450 7200
+F 0 "#PWR?" H 7450 7050 50  0001 C CNN
+F 1 "+3.3V" H 7450 7340 50  0000 C CNN
+F 2 "" H 7450 7200 50  0000 C CNN
+F 3 "" H 7450 7200 50  0000 C CNN
+	1    7450 7200
+	1    0    0    -1
+$EndComp
+$Comp
+L +3.3V #PWR?
+U 1 1 58F9E264
+P 14350 7800
+F 0 "#PWR?" H 14350 7650 50  0001 C CNN
+F 1 "+3.3V" H 14350 7940 50  0000 C CNN
+F 2 "" H 14350 7800 50  0000 C CNN
+F 3 "" H 14350 7800 50  0000 C CNN
+	1    14350 7800
+	1    0    0    -1
+$EndComp
+Wire Wire Line
+	13600 7850 14350 7850
+Text Label 13800 7750 0    60   ~ 0
+CANL
+Wire Wire Line
+	13800 7750 13600 7750
+Text Label 13800 7650 0    60   ~ 0
+CANH
+Wire Wire Line
+	13800 7650 13600 7650
+Wire Wire Line
+	14350 7850 14350 7800
+Text Label 9200 8350 0    60   ~ 0
+CAN_STB
+Wire Wire Line
+	9200 8350 9000 8350
+Text Label 13800 7550 0    60   ~ 0
+CAN_STB
+Wire Wire Line
+	13800 7550 13600 7550
+Text Notes 12500 7300 0    60   ~ 0
+CAN TRANCEIVER
 $EndSCHEMATC

Commit message: Finish wiring all base module components.
The schematic is still missing a supply, and there's a lot of
old stuff still lying around, so it's far from finished.
Connections:
- net labels added: EC_PWR, NUTR_ON, PH_ON, PMP_ON
- wire segments 205 -> 212
Other:
- note added: "PUMP CONTROLS"
- moved on the sheet: D?, Q?, R?
